File: hardware/design.kicad_pcb (KiCad board)
At the start: 2 copper layers, 94 x 94 mm, 23 parts, among them U1 ESP32-S3-Zero, U2 DIP-8, U3 RP2040, U4 AMT49413

Commit message: Minor pcb changes
Parts:
- D1, D2, D3, D4, D5, D6, D7, D8: footprint LED_SMD:LED_WS2812B_PLCC4_5.0x5.0mm_P3.2mm -> Library:LED_WS2812B_PLCC4_5.0x5.0mm_P3.2mm
Routing:
- net +5V: track 103.7 -> 107.3 mm
